Commit message: Update(farol_gazebo): changed altimeter frame_id to mimic real measurements

File: farol_gazebo/farol_vehicles/bluerov_heavy_vehicle/urdf/sensors.xacro (robot description, xacro)
@@ -30,11 +30,7 @@
   </xacro:default_dvl_bluerov_macro>
   <!-- Altimeter sensor 1 -->
-  <xacro:bluerov_altimeter namespace="${namespace}" parent_link="$(arg namespace)/base_link" suffix="1">
+  <xacro:bluerov_altimeter namespace="${namespace}" parent_link="$(arg namespace)/base_link" suffix="">
     <origin xyz="0.05 -0.07 -0.17" rpy="0 ${0.5*pi} 0"/>
   </xacro:bluerov_altimeter>
-  <!-- Altimeter sensor 2 -->
-  <!-- <xacro:bluerov_altimeter namespace="${namespace}" parent_link="$(arg namespace)/base_link" suffix="2">
-    <origin xyz="0.05 -0.07 -0.17" rpy="0 ${1.047197551} 0"/>
-  </xacro:bluerov_altimeter>      -->
   <!-- UDP camera -->
   <!-- <xacro:udp_camera_sensor_macro namespace="${namespace}" parent_link="$(arg namespace)/base_link" suffix=""

File: farol_gazebo/uuv_simulator/uuv_sensor_plugins/uuv_sensor_ros_plugins/urdf/altimeter_snippets.xacro (robot description, xacro)
@@ -93,5 +93,5 @@
                     <updateRate>15.0</updateRate>
                     <topicName>measurement/position</topicName>
-                    <frameName>${namespace}/altimeter${suffix}_link</frameName>
+                    <frameName>${namespace}_altimeter#</frameName>
                     <fov>${field_of_view}</fov>
                     <radiation>ultrasound</radiation>
