Commit message: Update(stuff): pushed the code because my pc might die :(

File: farol_gazebo/farol_vehicles/bluerov_heavy_vehicle/urdf/base.xacro (robot description, xacro)
@@ -13,5 +13,5 @@
     -->
   <!-- <xacro:property name="mass" value="15.5"/> -->
-  <xacro:property name="mass" value="10.5"/>
+  <xacro:property name="mass" value="11.5"/>
   <!-- Vehicle's bounding box: width, length, height -->
   <xacro:property name="x_size" value="0.448"/>
@@ -21,5 +21,5 @@
   <xacro:property name="z_size" value="0.2539"/>
   <!-- Volume -->
-  <xacro:property name="volume" value="0.011054"/>
+  <xacro:property name="volume" value="0.0115"/>
   <!-- Center of gravity -->
   <xacro:property name="cog" value="0 0 0"/>

File: farol_gazebo/farol_vehicles/bluerov_heavy_vehicle/urdf/gazebo.xacro (robot description, xacro)
@@ -22,19 +22,16 @@
           <type>fossen</type>
           <!-- Added mass: see p.28 in Berg2012 -->
+          <!-- Parameters in Sandøy, S. S. (2016). -->
           <added_mass>
-            27.08     0      0      0    0     0
-            0       25.952   0      0    0     0
-            0       0      29.9081  0    0     0
-            0       0      0        1    0     0
-            0       0      0        0    1     0
-            0       0      0        0    0     1
+            5.5     0      0        0    0     0
+            0       12.70  0        0    0     0
+            0       0      14.57    0    0     0
+            0       0      0        0.12 0     0
+            0       0      0        0    0.12  0
+            0       0      0        0    0     0.12
           </added_mass>
-          <!-- Linear damping: see p.31 in Berg2012 -->
-          <linear_damping>-0.1213 -1.1732 -1.1130 -0.5 -0.5 -0.5</linear_damping>
-          <!-- <linear_damping>-0.1213 -1.1732 -1.33 -0.5 -0.5 -0.5</linear_damping> -->
-          <!-- Non-linear damping: see p.30 in Berg2012 -->
-          <!--quadratic_damping>-18.18 -21.66 -36.99 -5.55 -5.55 -5.55</quadratic_damping-->
-          <!-- <quadratic_damping>-23.9000 -46.2700 -60.2780 -1 -1 -1</quadratic_damping> -->
-          <quadratic_damping>-23.9000 -46.2700 -50.2780 -1 -1 -1</quadratic_damping>
+          <!-- Parameters in Sandøy, S. S. (2016). -->
+          <linear_damping>-4.03  -6.22 -5.18 -0.07 -0.07 -0.07</linear_damping>
+          <quadratic_damping>-18.18 -21.66 -36.99 -1.55 -1.55 -1.55</quadratic_damping>
         </hydrodynamic_model>
       </link>
