Commit message: lalala

File: farol_gazebo/farol_vehicles/bluerov_heavy_vehicle/urdf/actuators.xacro (robot description, xacro)
@@ -10,17 +10,17 @@
     <!-- THRUSTER 1 - Horizontal-front starboard -->
     <xacro:thruster_macro robot_namespace="${namespace}" thruster_id="0">
-        <origin xyz="0.1355 -0.1 -0.0725" rpy="0 0 0.7853981634"/>
+        <origin xyz="0.14 -0.1 -0.0725" rpy="0 0 0.7853981634"/>
     </xacro:thruster_macro>
     <!-- THRUSTER 2 - Horizontal-front portside -->
     <xacro:thruster_macro robot_namespace="${namespace}" thruster_id="1">
-        <origin xyz="0.1355 0.1 -0.0725" rpy="0 0 -0.7853981634"/>
+        <origin xyz="0.14 0.1 -0.0725" rpy="0 0 -0.7853981634"/>
     </xacro:thruster_macro>
     <!-- THRUSTER 3 - Horizontal-back starboard -->
     <xacro:thruster_macro robot_namespace="${namespace}" thruster_id="2">
-        <origin xyz="-0.1475 -0.1 -0.0725" rpy="0 0 2.3561944902"/>
+        <origin xyz="-0.14 -0.1 -0.0725" rpy="0 0 2.3561944902"/>
     </xacro:thruster_macro>
     <!-- THRUSTER 4 - Horizontal-back portside -->
     <xacro:thruster_macro robot_namespace="${namespace}" thruster_id="3">
-        <origin xyz="-0.1475 0.1 -0.0725" rpy="0 0 -2.3561944902"/>
+        <origin xyz="-0.14 0.1 -0.0725" rpy="0 0 -2.3561944902"/>
     </xacro:thruster_macro>
     <!-- THRUSTER 5 - Vertical-front starboard -->

File: farol_gazebo/farol_vehicles/bluerov_heavy_vehicle/urdf/sensors.xacro (robot description, xacro)
@@ -27,9 +27,9 @@
     parent_link="${namespace}/base_link"
     inertial_reference_frame="${inertial_reference_frame}">
-    <origin xyz="0.05 0.07 -0.20" rpy="0 ${0.5*pi} 0"/>
+    <origin xyz="0.05 0.0 -0.20" rpy="0 ${0.5*pi} 0"/>
   </xacro:default_dvl_bluerov_macro>
   <!-- Altimeter sensor 1 -->
   <xacro:bluerov_altimeter namespace="${namespace}" parent_link="$(arg namespace)/base_link" suffix="">
-    <origin xyz="0.05 -0.07 -0.17" rpy="0 ${0.5*pi} 0"/>
+    <origin xyz="0.0 0.0 -0.22" rpy="0 ${0.5*pi} 0"/>
   </xacro:bluerov_altimeter>
   <!-- UDP camera -->
